Commit message: FLC open loop to ensure correct model

File: urdf/planar2dof.urdf (robot description, URDF)
Before this commit: robot planar2dof, 5 links, 4 joints
Links:
- link planar2dof/base_link: mass 1 -> 100
- link planar2dof/link_striker_ee: mass 0.0 -> 5.600

Commit message: Polynomial trajectory

File: urdf/planar2dof.urdf (robot description, URDF)
Before this commit: robot planar2dof, 5 links, 4 joints
Links:
- link planar2dof/link_striker_ee: mass 5.600 -> 1.0
